File: Hardware/Panel/Q Arduino Panel.brd (EAGLE design)
At the start: 116.8 x 129.5 mm, 84 parts, among them Q1 200mA/50V, Q2 200mA/50V, Q3 200mA/50V, Q4 200mA/50V, Q5 200mA/50V, Q6 200mA/50V, Q7 200mA/50V, Q8 200mA/50V, U1 ARDUINO UNO, U2 ARDUINO UNO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

Commit message: Adding panel
Routing:
- net CH64: track 10.2 -> 0.00 mm, vias 3 -> 0
- net CH63: track 10.2 -> 0.00 mm, vias 3 -> 0
- net CH62: track 10.2 -> 0.00 mm, vias 3 -> 0
- net CH61: track 10.2 -> 0.00 mm, vias 3 -> 0
- net CH60: track 10.2 -> 0.00 mm, vias 3 -> 0
- net CH59: track 10.2 -> 0.00 mm, vias 3 -> 0
- net CH58: track 10.2 -> 0.00 mm, vias 3 -> 0
- net CH57: track 10.2 -> 0.00 mm, vias 3 -> 0
- net 5V2: track 134.6 -> 129.8 mm
- net 5V1: track 134.6 -> 129.8 mm
- net 5V: track 134.6 -> 129.8 mm
- net 5V3: track 134.6 -> 129.8 mm
- net GND3: track 205.1 -> 201.4 mm
- net GND2: track 205.1 -> 201.4 mm
- net GND: track 205.1 -> 201.4 mm
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Other:
- board size 116.8 x 129.5 mm -> 124.5 x 142.2 mm
